File: pcbs/picopak/picopak.kicad_pcb (KiCad board)
At the start: 4 copper layers, 50 x 21 mm, 34 parts, among them J1 USB_B_Micro, J2 Conn_02x08_Odd_Even, J3 Conn_01x03_Female, J4 Conn_01x04_Female, SW1 sw, SW2 sw, SW3 sw, SW4 sw, U1 NCP1117-3.3_SOT223, U10 74LS245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

Commit message: Second PCB with errata fixed added
Parts:
- C4: footprint Capacitor_SMD:C_0805_2012Metric -> Capacitor_SMD:C_0402_1005Metric
- moved C5 6.74 mm to (205.2, 77.9), turned to 270 degrees
- moved R6 5.73 mm to (208.8, 75.1), turned to 90 degrees
- moved U1 2.60 mm to (199.6, 75.9)
- moved J4 1.50 mm to (206.8, 79.2)
Connections:
- J4 pad 1: GND -> I2C_SDA
- J4 pad 2: +3V3 -> I2C_SCLK
- J4 pad 3: I2C_SCLK -> +3V3
- J4 pad 4: I2C_SDA -> GND
- R6 pad 2: I2C_SDA -> I2C_SCLK
Routing:
- net GND: track 123.9 -> 157.4 mm
- net +3V3: track 106.8 -> 96.7 mm, vias 17 -> 16
- net I2C_SCLK: track 53.8 -> 61.6 mm, vias 5 -> 6
- net /USB_D+: track 21.7 -> 29.4 mm, vias 3 -> 5
- net /USB_D-: track 24.8 -> 32.0 mm
- net LS_DIR: track 42.0 -> 48.4 mm, vias 4 -> 7
- net VBUS: track 22.9 -> 25.7 mm
- net I2C_SDA: track 45.1 -> 43.3 mm
- net (no net): track 0.00 -> 0.97 mm, vias 0 -> 1
- net SPGM: track 6.83 -> 7.56 mm
Other:
- outline, holes or cut-outs redrawn
- board text added: "GND"
- board text added: "PicoPak for Psion V1.1 August 2021 menadue@gmail.com"
- board text added: "SCLK"
- board text removed: "G"
- board text removed: "PicoPak for Psion July 2021 menadue@gmail.com"
- board text removed: "SLK"

Commit message: Added RUN jumper for drag-drop upgrade, SWD pads moved
Parts:
- added JP1: Jumper_NO_Small, Jumper:SolderJumper-2_P1.3mm_Open_Pad1.0x1.5mm, F.Cu at (203.9, 74.4)
- added R7: 1k, Capacitor_SMD:C_0402_1005Metric, F.Cu at (203.7, 77.3)
- moved J3 15.6 mm to (162.2, 71.9)
Routing:
- net /SWCLK: track 5.42 -> 22.2 mm, vias 0 -> 2
- net /SWD: track 7.67 -> 21.2 mm, vias 0 -> 2
- net GND: track 157.4 -> 167.7 mm
- net /QSPI_SS: track 24.2 -> 29.7 mm
- net Net-(JP1-Pad1): track 0.00 -> 1.82 mm
- net SD6: vias 2 -> 1
- net +3V3: vias 16 -> 17
Other:
- board text added: "PicoPak for Psion V1.2 Sept 2021 menadue@gmail.com"
- board text removed: "GND"
- board text removed: "PicoPak for Psion V1.1 August 2021 menadue@gmail.com"

Commit message: V1_2 PCB laid out
Parts:
- added D1: PMEG3010ER, Diode_SMD:D_SOD-123, B.Cu at (206.2, 84.6)
- added J5: Conn_01x02_Female, Connector_PinHeader_1.00mm:PinHeader_1x02_P1.00mm_Vertical_SMD_Pin1Left, B.Cu at (162.6, 88.2)
- added R8: R_Small, Capacitor_SMD:C_0402_1005Metric, B.Cu at (163.4, 82.3)
- added R9: R_Small, Capacitor_SMD:C_0402_1005Metric, B.Cu at (161.9, 82.1)
- added TR1: Si2302CDS-n-channel, Package_TO_SOT_SMD:SOT-23, B.Cu at (162.4, 85.1)
- moved R2 2.91 mm to (201.6, 80.1), turned to 180 degrees
Connections:
- C1 pad 1: VBUS -> Net-(C1-Pad1)
- J1 pad 1: VBUS -> Net-(D1-Pad2)
- U1 pad 3: VBUS -> Net-(C1-Pad1)
- U3 pad 41: (no net) -> BATSENSE
Routing:
- net Net-(C1-Pad1): track 0.00 -> 70.4 mm, vias 0 -> 3
- net BATSENSE: track 0.00 -> 33.4 mm, vias 0 -> 2
- net VBUS: track 25.7 -> 0.00 mm, vias 1 -> 0
- net Net-(D1-Pad2): track 0.00 -> 14.8 mm, vias 0 -> 1
- net +3V3: track 96.7 -> 101.9 mm
- net Net-(J5-Pad2): track 0.00 -> 4.95 mm
- net LS_DIR: track 48.4 -> 51.3 mm
- net Net-(J5-Pad1): track 0.00 -> 2.78 mm
- net GND: track 167.7 -> 169.8 mm
- net /QSPI_SS: track 29.7 -> 30.5 mm
Other:
- board text added: "LOAD"
- board text added: "VBAT"
- board text added: "VLCD"

Commit message: Updates. Archive file for PCB
Parts:
- added M1: Si2301 P chan, Package_TO_SOT_SMD:SOT-23, B.Cu at (166.0, 84.1)
- added R10: 10k, Capacitor_SMD:C_0402_1005Metric, B.Cu at (161.4, 87.4)
- added R11: 100k, Capacitor_SMD:C_0402_1005Metric, B.Cu at (165.8, 87.2)
- moved TR1 0.40 mm to (162.4, 84.7)
Connections:
- TR1 pad 1: Net-(J5-Pad1) -> Net-(R10-Pad1)
- TR1 pad 2: Net-(C1-Pad1) -> GND
- TR1 pad 3: Net-(J5-Pad2) -> Net-(M1-Pad1)
Routing:
- net Net-(J5-Pad2): track 4.95 -> 9.81 mm
- net Net-(M1-Pad1): track 0.00 -> 3.74 mm
- net Net-(C1-Pad1): track 70.4 -> 66.7 mm
- net GND: track 169.8 -> 172.5 mm
- net Net-(J5-Pad1): track 2.78 -> 0.95 mm
- net Net-(R10-Pad1): track 0.00 -> 0.87 mm

Commit message: Update
Other:
- board text added: "PicoPak for Psion Nov 2021 V1.3 menadue@gmail.com"
- board text removed: "PicoPak for Psion V1.2 Sept 2021 menadue@gmail.com"
Changed lines of the file:
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@@
       (drillshape 0)
       (scaleselection 1)
-      (outputdirectory "fab3/"))
+      (outputdirectory "fab1_3/"))
   )
   (net 0 "")
@@
     (add_net /QSPI_SD3)
     (add_net /QSPI_SS)
-    (add_net /RUN)
     (add_net /SWCLK)
     (add_net /SWD)
@@
     (add_net "Net-(C3-Pad1)")
     (add_net "Net-(D1-Pad2)")
-    (add_net "Net-(J2-Pad1)")
-    (add_net "Net-(J2-Pad2)")
     (add_net "Net-(J5-Pad1)")
     (add_net "Net-(J5-Pad2)")
@@
     (add_net "Net-(R3-Pad2)")
     (add_net "Net-(R4-Pad2)")
-    (add_net "Net-(U3-Pad35)")
-    (add_net "Net-(U3-Pad36)")
-    (add_net "Net-(U3-Pad37)")
-    (add_net "Net-(U9-Pad11)")
-    (add_net "Net-(U9-Pad12)")
-    (add_net "Net-(U9-Pad13)")
-    (add_net "Net-(U9-Pad7)")
-    (add_net "Net-(U9-Pad8)")
-    (add_net "Net-(U9-Pad9)")
-    (add_net "Net-(XS1-Pad9)")
     (add_net P_SCLK)
     (add_net P_SD0)
@@
     (tags SOT-23)
     (attr smd)
-    (fp_text reference M1 (at 0 2.5) (layer B.SilkS)
-      (effects (font (size 1 1) (thickness 0.15)) (justify mirror))
+    (fp_text reference M1 (at 1.7 1.3) (layer B.SilkS)
+      (effects (font (size 0.75 0.75) (thickness 0.1)) (justify mirror))
     )
     (fp_text value "Si2301 P chan" (at 0 -2.5) (layer B.Fab)
@@
     (tags capacitor)
     (attr smd)
-    (fp_text reference R11 (at 0 1.17 270) (layer B.SilkS)
-      (effects (font (size 1 1) (thickness 0.15)) (justify mirror))
+    (fp_text reference R11 (at 0 1.8 270) (layer B.SilkS)
+      (effects (font (size 0.7 1) (thickness 0.15)) (justify mirror))
     )
     (fp_text value 100k (at 0 -1.17 270) (layer B.Fab)
@@
     (tags capacitor)
     (attr smd)
-    (fp_text reference R10 (at 0 1.17 90) (layer B.SilkS)
-      (effects (font (size 1 1) (thickness 0.15)) (justify mirror))
+    (fp_text reference R10 (at 0.2 1 90) (layer B.SilkS)
+      (effects (font (size 0.7 1) (thickness 0.15)) (justify mirror))
     )
     (fp_text value 10k (at 0 -1.17 90) (layer B.Fab)
@@
     (tags capacitor)
     (attr smd)
-    (fp_text reference R9 (at 2 0 90) (layer B.SilkS)
-      (effects (font (size 1 1) (thickness 0.15)) (justify mirror))
+    (fp_text reference R9 (at 1.7 0.5 90) (layer B.SilkS)
+      (effects (font (size 0.75 0.75) (thickness 0.1)) (justify mirror))
     )
     (fp_text value R_Small (at 0 -1.17 90) (layer B.Fab)
@@
     (tags capacitor)
     (attr smd)
-    (fp_text reference R8 (at 2 0.1 90) (layer B.SilkS)
-      (effects (font (size 1 1) (thickness 0.15)) (justify mirror))
+    (fp_text reference R8 (at 1.9 0.9 90) (layer B.SilkS)
+      (effects (font (size 0.75 0.75) (thickness 0.1)) (justify mirror))
     )
     (fp_text value R_Small (at 0 -1.17 90) (layer B.Fab)
@@
     (attr smd)
     (fp_text reference TR1 (at -1.7 -2.8 90) (layer B.SilkS)
-      (effects (font (size 1 1) (thickness 0.15)) (justify mirror))
+      (effects (font (size 0.75 0.75) (thickness 0.1)) (justify mirror))
     )
     (fp_text value Si2302CDS-n-channel (at 0 -2.5) (layer B.Fab)
@@
     (tags "Surface mounted pin header SMD 1x02 1.00mm single row style1 pin1 left")
     (attr smd)
-    (fp_text reference J5 (at -1.3 -0.5) (layer B.SilkS)
+    (fp_text reference J5 (at 1.6 -1.5) (layer B.SilkS)
       (effects (font (size 0.75 0.75) (thickness 0.15)) (justify mirror))
     )
@@
     (tags "solder jumper open")
     (attr virtual)
-    (fp_text reference JP1 (at 0.624999 -1.8 270) (layer F.SilkS)
+    (fp_text reference JP1 (at 2.724999 0 270) (layer F.SilkS)
       (effects (font (size 0.75 0.75) (thickness 0.15)))
     )
@@
     (tags "Surface mounted pin header SMD 1x03 1.00mm single row style1 pin1 left")
     (attr smd)
-    (fp_text reference J3 (at -2.7 0) (layer B.SilkS)
-      (effects (font (size 1 1) (thickness 0.15)) (justify mirror))
+    (fp_text reference J3 (at -1.6 2.2) (layer B.SilkS)
+      (effects (font (size 0.75 0.75) (thickness 0.1)) (justify mirror))
     )
     (fp_text value Conn_01x03_Female (at 0 -2.56) (layer B.Fab)
@@
     (tags capacitor)
     (attr smd)
-    (fp_text reference C7 (at 2.5 0.1) (layer B.SilkS)
+    (fp_text reference C7 (at 0.1 1.1) (layer B.SilkS)
       (effects (font (size 0.75 0.75) (thickness 0.15)) (justify mirror))
     )
@@
     (tags capacitor)
     (attr smd)
-    (fp_text reference C8 (at -0.2 -2.8) (layer B.SilkS)
-      (effects (font (size 1 1) (thickness 0.15)) (justify mirror))
+    (fp_text reference C8 (at 1.7 0.5) (layer B.SilkS)
+      (effects (font (size 0.75 0.75) (thickness 0.1)) (justify mirror))
     )
     (fp_text value 1u (at 0 -1.17) (layer B.Fab)
@@
     (tags capacitor)
     (attr smd)
-    (fp_text reference C10 (at 0.3 -3.1) (layer B.SilkS)
-      (effects (font (size 1 1) (thickness 0.15)) (justify mirror))
+    (fp_text reference C10 (at 0.1 -0.9) (layer B.SilkS)
+      (effects (font (size 0.75 0.75) (thickness 0.1)) (justify mirror))
     )
     (fp_text value 1u (at 0 -1.17) (layer B.Fab)
@@
     (tags capacitor)
     (attr smd)
-    (fp_text reference C15 (at 0.8 -3.1) (layer B.SilkS)
-      (effects (font (size 1 1) (thickness 0.15)) (justify mirror))
+    (fp_text reference C15 (at 0 -1) (layer B.SilkS)
+      (effects (font (size 0.75 0.75) (thickness 0.1)) (justify mirror))
     )
     (fp_text value 100n (at 0 -1.17) (layer B.Fab)
@@
     (tags capacitor)
     (attr smd)
-    (fp_text reference R15 (at 2 0.9) (layer B.SilkS)
-      (effects (font (size 1 1) (thickness 0.15)) (justify mirror))
+    (fp_text reference R15 (at -0.4 -0.7) (layer B.SilkS)
+      (effects (font (size 0.75 0.75) (thickness 0.1)) (justify mirror))
     )
     (fp_text value R_Small (at 0 -1.17) (layer B.Fab)
@@
     (tags capacitor)
     (attr smd)
-    (fp_text reference R4 (at -2.7 0) (layer B.SilkS)
+    (fp_text reference R4 (at -1.9 -0.1) (layer B.SilkS)
       (effects (font (size 0.75 0.75) (thickness 0.15)) (justify mirror))
     )
@@
     (tags capacitor)
     (attr smd)
-    (fp_text reference R3 (at -2.4 -0.1) (layer B.SilkS)
+    (fp_text reference R3 (at -1.8 -0.1) (layer B.SilkS)
       (effects (font (size 0.75 0.75) (thickness 0.15)) (justify mirror))
     )
@@
   (gr_line (start 174 71) (end 177 71) (layer Edge.Cuts) (width 0.05))
   (gr_line (start 174 69) (end 174 71) (layer Edge.Cuts) (width 0.05))
-  (gr_text "PicoPak for Psion V1.2\nSept 2021\nmenadue@gmail.com" (at 166.4 85.9 90) (layer B.SilkS)
-    (effects (font (size 0.75 0.75) (thickness 0.15)) (justify right mirror))
+  (gr_text "PicoPak for Psion\nNov 2021  V1.3\nmenadue@gmail.com" (at 166.5 71.4 90) (layer B.SilkS)
+    (effects (font (size 0.75 0.75) (thickness 0.15)) (justify left mirror))
   )
   (gr_text SCLK (at 162 74.5) (layer B.SilkS)
