File: pcbs/picopak/_autosave-picopak.kicad_pcb (KiCad board)
At the start: 4 copper layers, 50 x 21 mm, 44 parts, among them J1 USB_B_Micro, J2 Conn_02x08_Odd_Even, J3 Conn_01x03_Female, J4 Conn_01x04_Female, J5 Conn_01x02_Female, M1 Si2301 P chan, SW1 sw, SW2 sw, SW3 sw, SW4 sw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

Commit message: "Update"
Parts:
- R8, R9: value 1m -> 1M
Changed lines of the file:
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@@
 			)
 		)
-		(property "Value" "1m"
+		(property "Value" "1M"
 			(at 0 -1.17 90)
 			(layer "B.Fab")
@@
 			)
 		)
-		(property "Value" "1m"
+		(property "Value" "1M"
 			(at 0 -1.17 90)
 			(layer "B.Fab")
